File: KiCad_VFD_clock_driver/VFD_clock_driver.sch (KiCad schematic (older format))
At the start: 43 parts

Commit message: Final driver schematic
Final driver PCB schematic
Parts:
- removed C?: 1F GoldCap, symbol Device:CP
- added BT1: RTC li-ion, Battery:BatteryHolder_Seiko_MS621F, symbol Device:Battery_Cell
- added C10, C11, C12, C5, C7, C8, C9: 100nF, Capacitor_SMD:C_1206_3216Metric, symbol Device:C_Small
- added D3: LED, Diode_SMD:D_1206_3216Metric_Pad1.42x1.75mm_HandSolder, symbol Device:LED_Small
- added J2: SWD, Connector_PinHeader_2.54mm:PinHeader_1x04_P2.54mm_Horizontal, symbol Connector:Conn_01x04_Male
- added R10: 4.7K, Resistor_SMD:R_1206_3216Metric, symbol Device:R_Small
- added R27, R8: 10K, Resistor_SMD:R_1206_3216Metric, symbol Device:R_Small
- added R7: 1.5K, Resistor_SMD:R_1206_3216Metric, symbol Device:R_Small
- added SW1: RESET, Button_Switch_SMD:SW_SPST_TL3342, symbol Switch:SW_Push
- added SW2: SELECT, Button_Switch_THT:SW_Tactile_SPST_Angled_PTS645Vx83-2LFS, symbol Switch:SW_Push
- added SW3: PLUS, Button_Switch_THT:SW_Tactile_SPST_Angled_PTS645Vx83-2LFS, symbol Switch:SW_Push
- added SW4: MINUS, Button_Switch_THT:SW_Tactile_SPST_Angled_PTS645Vx83-2LFS, symbol Switch:SW_Push
- added U5: DHT11, Sensor:Aosong_DHT11_5.5x12.0_P2.54mm, symbol Sensor:DHT11
- J3, J4: renamed from J?; footprint (none) -> Connector_PinSocket_2.54mm:PinSocket_1x08_P2.54mm_Vertical
- L1: renamed from L?; footprint (none) -> Inductor_SMD:L_6.3x6.3_H3
- R5: renamed from R?; value 100R -> 1K
- gave numbers to parts that had none: 38
Connections:
- net labels added: BUTTON_MINUS, BUTTON_PLUS, BUTTON_SELECT, DHT_interface, USART_RX, USART_TX, VBAT
- wire segments 198 -> 257
- no-connect marks 3 -> 8
Other:
- note added: "3.3V"
- note added: "DHT11 humidity sensor"
- note added: "DS18B20 temperature sensor"
- note added: "DS3231 RTC"
- note added: "GND"
- note added: "MCU power filtering capactiros"
- note added: "STM32F103C8T6 microcontroller"
- note added: "SWCLK"
- note added: "SWDIO"
- note added: "VFD voltage converters"
- note added: "power supply"
- note added: "user inteface buttons"
- moved on the sheet: J3, J4, R11, R12, R13, R14, R15, R16, R17, R18, R19, R20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

Commit message: Buzzer and additional inputs
+ added buzzer with circuitry
+ SQW and UART connected to MCU
Parts:
- added BZ1: Buzzer, Buzzer_Beeper:Buzzer_12x9.5RM7.6, symbol Device:Buzzer
- added C13: 47uF, Capacitor_SMD:CP_Elec_5x4.4, symbol Device:CP_Small
- added C14: 100nF, Capacitor_SMD:C_1206_3216Metric, symbol Device:C_Small
- added J5: UART, Connector_PinHeader_2.54mm:PinHeader_1x04_P2.54mm_Horizontal, symbol Connector:Conn_01x04_Male
- added Q1: BC547, Package_TO_SOT_THT:TO-92_Inline, symbol Transistor_BJT:BC547
- added R28: 1K, Resistor_SMD:R_1206_3216Metric, symbol Device:R_Small
- added R29: 10K, Resistor_SMD:R_1206_3216Metric, symbol Device:R_Small
Connections:
- net +3V3: now also J5.4 (Pin_4)
- net GND: now also C13.2, C14.1, J5.1 (Pin_1), Q1.3 (E)
- net SQW: now also U6.5 (PD0)
- net BUZZER: now reaches U6.29 (PA8)
- net BUZZER: now also R29.1
- net VIN: now reaches C1.1, C2.1, J1.1, L1.1, U2.4 (EN), U2.5 (VIN), U3.3 (VI)
- net VIN: now also C13.1, C14.2, R28.2
- net USART_RX: no longer names the net of U6.31 (PA10)
- net USART_RX: now also J5.2 (Pin_2)
- net USART_TX: no longer names the net of U6.30 (PA9)
- net USART_TX: now also J5.3 (Pin_3)
- new net: BZ1.1 (-), R28.1
- new net: BZ1.2 (+), Q1.1 (C)
- new net: Q1.2 (B), R29.2
- no-connect marks 8 -> 10
Other:
- note added: "BUZZER"
- note added: "RX"
- note added: "TX"
Changed lines of the file:
@@
 Connection ~ 2350 1100
-Wire Wire Line
-	2350 1100 2900 1100
 Wire Wire Line
 	1600 1300 1650 1300
@@
 Text Label 8550 8250 2    50   ~ 0
 DHT_interface
-Text Label 9850 8250 0    50   ~ 0
-USART_TX
-Text Label 9850 8350 0    50   ~ 0
-USART_RX
-Wire Notes Line
-	6850 9650 11450 9650
 Text Notes 6800 5300 0    100  ~ 0
 STM32F103C8T6 microcontroller
-Wire Notes Line
-	6800 5150 6800 9700
 Wire Notes Line
 	6800 5350 11450 5350
@@
 NoConn ~ 9850 8550
 NoConn ~ 9850 8450
-NoConn ~ 9850 8150
 NoConn ~ 8550 8550
 Wire Wire Line
@@
 Wire Notes Line
 	10050 6700 10050 5350
+$Comp
+L Connector:Conn_01x04_Male J5
+U 1 1 5FCADB4E
+P 10700 7750
+F 0 "J5" H 10550 7650 50  0000 C CNN
+F 1 "UART" H 10550 7750 50  0000 C CNN
+F 2 "Connector_PinHeader_2.54mm:PinHeader_1x04_P2.54mm_Horizontal" H 10700 7750 50  0001 C CNN
+F 3 "~" H 10700 7750 50  0001 C CNN
+	1    10700 7750
+	-1   0    0    1
+$EndComp
+$Comp
+L power:+3.3V #PWR03
+U 1 1 5FCADB54
+P 10450 7500
+F 0 "#PWR03" H 10450 7350 50  0001 C CNN
+F 1 "+3.3V" H 10465 7673 50  0000 C CNN
+F 2 "" H 10450 7500 50  0001 C CNN
+F 3 "" H 10450 7500 50  0001 C CNN
+	1    10450 7500
+	1    0    0    -1
+$EndComp
+Wire Wire Line
+	10500 7550 10450 7550
+Wire Wire Line
+	10450 7550 10450 7500
+$Comp
+L power:GND #PWR04
+U 1 1 5FCADB5C
+P 10450 7900
+F 0 "#PWR04" H 10450 7650 50  0001 C CNN
+F 1 "GND" H 10455 7727 50  0000 C CNN
+F 2 "" H 10450 7900 50  0001 C CNN
+F 3 "" H 10450 7900 50  0001 C CNN
+	1    10450 7900
+	1    0    0    -1
+$EndComp
+Wire Wire Line
+	10500 7850 10450 7850
+Wire Wire Line
+	10450 7850 10450 7900
+Text Notes 10950 7550 0    50   ~ 0
+3.3V
+Text Notes 10950 7850 0    50   ~ 0
+GND
+Text Notes 10950 7650 0    50   ~ 0
+TX
+Text Notes 10950 7750 0    50   ~ 0
+RX
+Wire Wire Line
+	9850 8250 10200 8250
+Wire Wire Line
+	10200 8250 10200 7650
+Wire Wire Line
+	10200 7650 10500 7650
+Wire Wire Line
+	10500 7750 10250 7750
+Wire Wire Line
+	10250 7750 10250 8350
+Wire Wire Line
+	10250 8350 9850 8350
+Text Label 8550 6650 2    50   ~ 0
+SQW
+Wire Notes Line
+	6800 9650 11450 9650
+Wire Notes Line
+	6800 9650 6800 5150
+$Comp
+L Device:Buzzer BZ1
+U 1 1 5FDCF8D8
+P 3550 7400
+F 0 "BZ1" V 3601 7213 50  0000 R CNN
+F 1 "Buzzer" V 3510 7213 50  0000 R CNN
+F 2 "Buzzer_Beeper:Buzzer_12x9.5RM7.6" V 3525 7500 50  0001 C CNN
+F 3 "~" V 3525 7500 50  0001 C CNN
+	1    3550 7400
+	0    -1   -1   0
+$EndComp
+$Comp
+L Transistor_BJT:BC547 Q1
+U 1 1 5FDD00A6
+P 4350 7600
+F 0 "Q1" H 4541 7646 50  0000 L CNN
+F 1 "BC547" H 4541 7555 50  0000 L CNN
+F 2 "Package_TO_SOT_THT:TO-92_Inline" H 4550 7525 50  0001 L CIN
+F 3 "http://www.fairchildsemi.com/ds/BC/BC547.pdf" H 4350 7600 50  0001 L CNN
+	1    4350 7600
+	0    -1   -1   0
+$EndComp
+$Comp
+L Device:CP_Small C13
+U 1 1 5FDE4E41
+P 1800 7700
+F 0 "C13" H 1888 7746 50  0000 L CNN
+F 1 "47uF" H 1888 7655 50  0000 L CNN
+F 2 "Capacitor_SMD:CP_Elec_5x4.4" H 1800 7700 50  0001 C CNN
+F 3 "~" H 1800 7700 50  0001 C CNN
+	1    1800 7700
+	1    0    0    -1
+$EndComp
+$Comp
+L Device:C_Small C14
+U 1 1 5FE1EBEE
+P 2500 7700
+F 0 "C14" H 2592 7746 50  0000 L CNN
+F 1 "100nF" H 2592 7655 50  0000 L CNN
+F 2 "Capacitor_SMD:C_1206_3216Metric" H 2500 7700 50  0001 C CNN
+F 3 "~" H 2500 7700 50  0001 C CNN
+	1    2500 7700
+	-1   0    0    1
+$EndComp
+Wire Wire Line
+	1800 7600 1800 7500
+Wire Wire Line
+	1800 7500 2500 7500
+Wire Wire Line
+	2500 7500 2500 7600
+Wire Wire Line
+	2500 7500 3050 7500
+Connection ~ 2500 7500
+Wire Wire Line
+	3650 7500 4150 7500
+$Comp
+L Device:R_Small R29
+U 1 1 5FEF3892
+P 4350 8050
+F 0 "R29" H 4291 8004 50  0000 R CNN
+F 1 "10K" H 4291 8095 50  0000 R CNN
+F 2 "Resistor_SMD:R_1206_3216Metric" H 4350 8050 50  0001 C CNN
+F 3 "~" H 4350 8050 50  0001 C CNN
+	1    4350 8050
+	-1   0    0    1
+$EndComp
+Wire Wire Line
+	4350 7950 4350 7800
+Wire Wire Line
+	4350 8150 4350 8400
+Wire Wire Line
+	1800 7500 1450 7500
+Wire Wire Line
+	1450 7500 1450 7400
+Connection ~ 1800 7500
+Wire Wire Line
+	2350 1100 2350 950
+Text Label 2350 950  0    50   ~ 0
+VIN
+Wire Wire Line
+	2350 1100 2900 1100
+Text Label 1450 7400 0    50   ~ 0
+VIN
+$Comp
+L Device:R_Small R28
+U 1 1 6001400B
+P 3150 7500
+F 0 "R28" V 2954 7500 50  0000 C CNN
+F 1 "1K" V 3045 7500 50  0000 C CNN
+F 2 "Resistor_SMD:R_1206_3216Metric" H 3150 7500 50  0001 C CNN
+F 3 "~" H 3150 7500 50  0001 C CNN
+	1    3150 7500
+	0    1    1    0
+$EndComp
+Wire Wire Line
+	3250 7500 3450 7500
+Wire Wire Line
+	4550 7500 4900 7500
+$Comp
+L power:GND #PWR07
+U 1 1 600534C1
+P 4900 7500
+F 0 "#PWR07" H 4900 7250 50  0001 C CNN
+F 1 "GND" H 4905 7327 50  0000 C CNN
+F 2 "" H 4900 7500 50  0001 C CNN
+F 3 "" H 4900 7500 50  0001 C CNN
+	1    4900 7500
+	0    -1   -1   0
+$EndComp
+Wire Wire Line
+	2500 7800 2500 8050
+Wire Wire Line
+	1800 7800 1800 8050
+$Comp
+L power:GND #PWR05
+U 1 1 600E95C9
+P 1800 8050
+F 0 "#PWR05" H 1800 7800 50  0001 C CNN
+F 1 "GND" H 1805 7877 50  0000 C CNN
+F 2 "" H 1800 8050 50  0001 C CNN
+F 3 "" H 1800 8050 50  0001 C CNN
+	1    1800 8050
+	1    0    0    -1
+$EndComp
+$Comp
+L power:GND #PWR06
+U 1 1 600FEB39
+P 2500 8050
+F 0 "#PWR06" H 2500 7800 50  0001 C CNN
+F 1 "GND" H 2505 7877 50  0000 C CNN
+F 2 "" H 2500 8050 50  0001 C CNN
+F 3 "" H 2500 8050 50  0001 C CNN
+	1    2500 8050
+	1    0    0    -1
+$EndComp
+Text Label 4350 8400 0    50   ~ 0
+BUZZER
+Text Label 9850 8150 0    50   ~ 0
+BUZZER
+NoConn ~ 8550 7150
+NoConn ~ 8550 7050
+NoConn ~ 8550 6750
+Wire Notes Line
+	1050 6900 5500 6900
+Text Notes 1050 6850 0    100  ~ 0
+BUZZER
+Wire Notes Line
+	1050 6700 5500 6700
+Wire Notes Line
+	1050 6700 1050 9350
+Wire Notes Line
+	5500 6700 5500 9350
+Wire Notes Line
+	5500 9350 1050 9350
 $EndSCHEMATC

Commit message: Power supply section in PCB
Parts:
- D2: footprint Diode_SMD:D_SMC -> Diode_SMD:D_SMA
- U2: footprint Package_TO_SOT_SMD:SOT-23-6 -> Package_TO_SOT_SMD:SOT-23-5_HandSoldering
Changed lines of the file:
@@
 F 0 "U2" H 3700 2125 50  0000 C CNN
 F 1 "SX1308" H 3700 2034 50  0000 C CNN
-F 2 "Package_TO_SOT_SMD:SOT-23-6" H 3700 2100 50  0001 C CNN
+F 2 "Package_TO_SOT_SMD:SOT-23-5_HandSoldering" H 3700 2100 50  0001 C CNN
 F 3 "" H 3700 2100 50  0001 C CNN
 	1    3700 1700
@@
 F 0 "D2" H 4400 895 50  0000 C CNN
 F 1 "SS34" H 4400 986 50  0000 C CNN
-F 2 "Diode_SMD:D_SMC" V 4400 1100 50  0001 C CNN
+F 2 "Diode_SMD:D_SMA" V 4400 1100 50  0001 C CNN
 F 3 "~" V 4400 1100 50  0001 C CNN
 	1    4400 1100

Commit message: VFD tube power connector on BCB
Parts:
- added J6: VFD display power, Connector_PinSocket_2.54mm:PinSocket_1x04_P2.54mm_Vertical, symbol Connector:Conn_01x04_Female
Connections:
- net +3V3: now also J6.2 (Pin_2)
- net GND: now also J6.1 (Pin_1), J6.4 (Pin_4)
- net VIN: now also J6.3 (Pin_3)
Changed lines of the file:
@@
 Wire Notes Line
 	5500 9350 1050 9350
+$Comp
+L Connector:Conn_01x04_Female J6
+U 1 1 5FB809FA
+P 1950 3050
+F 0 "J6" H 1978 3026 50  0000 L CNN
+F 1 "VFD display power" H 1978 2935 50  0000 L CNN
+F 2 "Connector_PinSocket_2.54mm:PinSocket_1x04_P2.54mm_Vertical" H 1950 3050 50  0001 C CNN
+F 3 "~" H 1950 3050 50  0001 C CNN
+	1    1950 3050
+	1    0    0    -1
+$EndComp
+$Comp
+L power:GND #PWR0124
+U 1 1 5FB854C8
+P 1600 3300
+F 0 "#PWR0124" H 1600 3050 50  0001 C CNN
+F 1 "GND" H 1605 3127 50  0000 C CNN
+F 2 "" H 1600 3300 50  0001 C CNN
+F 3 "" H 1600 3300 50  0001 C CNN
+	1    1600 3300
+	1    0    0    -1
+$EndComp
+Wire Wire Line
+	1750 3250 1600 3250
+Wire Wire Line
+	1600 3250 1600 3300
+Wire Wire Line
+	1750 2950 1600 2950
+Wire Wire Line
+	1600 2950 1600 3250
+Connection ~ 1600 3250
+$Comp
+L power:+3.3V #PWR0125
+U 1 1 5FC0E222
+P 1300 3000
+F 0 "#PWR0125" H 1300 2850 50  0001 C CNN
+F 1 "+3.3V" H 1315 3173 50  0000 C CNN
+F 2 "" H 1300 3000 50  0001 C CNN
+F 3 "" H 1300 3000 50  0001 C CNN
+	1    1300 3000
+	1    0    0    -1
+$EndComp
+Text Label 1300 3150 2    50   ~ 0
+VIN
+Wire Wire Line
+	1300 3050 1300 3000
+Wire Wire Line
+	1300 3050 1750 3050
+Wire Wire Line
+	1300 3150 1750 3150
 $EndSCHEMATC

Commit message: External PCB for VFD tube and H-brigde
+ additional PCB for VFD tube with H-bridge
Parts:
- added C15: 47uF, Capacitor_SMD:CP_Elec_5x4.4, symbol Device:CP_Small
- added C16: 100nF, Capacitor_SMD:C_1206_3216Metric, symbol Device:C_Small
- added J7: VFD display driver, Connector_PinHeader_2.54mm:PinHeader_1x04_P2.54mm_Vertical, symbol Connector:Conn_01x04_Male
- added J8: Segments inputs, Connector_PinHeader_2.54mm:PinHeader_1x08_P2.54mm_Vertical, symbol Connector:Conn_01x08_Male
- added J9: Multiplexer inputs, Connector_PinHeader_2.54mm:PinHeader_1x08_P2.54mm_Vertical, symbol Connector:Conn_01x08_Male
- added Q2: BC547, Package_TO_SOT_THT:TO-92_Inline, symbol Transistor_BJT:BC547
- added R30: 1K, Resistor_SMD:R_1206_3216Metric, symbol Device:R_Small
- added R31: 10K, Resistor_SMD:R_1206_3216Metric, symbol Device:R_Small
- added RV2: 1K, Potentiometer_THT:Potentiometer_Piher_PT-6-V_Vertical_Hole, symbol Device:R_POT_Small
- added U10: L293, Package_DIP:DIP-16_W7.62mm, symbol Driver_Motor:L293
- added U9: AMS1117-5.0, Package_TO_SOT_SMD:SOT-223-3_TabPin2, symbol Regulator_Linear:AMS1117-5.0
- added VFD1: IV-18, WK_lib:IV-18, symbol WK_lib:IV-18
- J6: value VFD display power -> VFD display driver
Connections:
- net GND: no longer J6.1 (Pin_1)
- net VFD_AC: now reaches U6.38 (PA15)
- net VFD_AC: now also J6.1 (Pin_1)
- new net: U10.6 (2Y), VFD1.1 (FILAMENT+)
- new net: J8.2 (Pin_2), VFD1.10 (B)
- new net: J8.6 (Pin_6), VFD1.11 (F)
- new net: J8.1 (Pin_1), VFD1.12 (A)
- new net: RV2.3, VFD1.13 (FILAMENT-)
- new net: J9.1 (Pin_1), VFD1.15 (L1)
- new net: J9.3 (Pin_3), VFD1.16 (L3)
- new net: J9.5 (Pin_5), VFD1.17 (L5)
- new net: J9.8 (Pin_8), VFD1.18 (L8)
- new net: J9.7 (Pin_7), VFD1.19 (L7)
- new net: J8.8 (Pin_8), VFD1.2 (DP)
- new net: J9.6 (Pin_6), VFD1.20 (L6)
- new net: J9.4 (Pin_4), VFD1.21 (L4)
- new net: J9.2 (Pin_2), VFD1.22 (L2)
- new net: J8.4 (Pin_4), VFD1.3 (D)
- new net: J8.3 (Pin_3), VFD1.4 (C)
- new net: J8.5 (Pin_5), VFD1.5 (E)
- new net: J8.7 (Pin_7), VFD1.9 (G)
- new net: C15.2, C16.2, J7.1 (Pin_1), Q2.3 (E), U10.12 (GND), U10.13 (GND), U10.4 (GND), U10.5 (GND), U9.1 (GND)
- new net: C15.1, C16.1, U10.8 (VCC2), U9.2 (VO)
- new net: J7.2 (Pin_2), U9.3 (VI)
- new net: RV2.2, U10.3 (1Y)
- new net: J7.3 (Pin_3), R31.2, U10.1 (EN1,2), U10.16 (VCC1)
- new net: J7.4 (Pin_4), R30.1, U10.2 (1A)
- new net: Q2.1 (C), R31.1, U10.7 (2A)
- new net: Q2.2 (B), R30.2
- no-connect marks 10 -> 16
Other:
- note added: "VFD display and driver"
- note added: "VFD_AC"
- note added: "VIN"
- moved on the sheet: BT1, BZ1, C1, C10, C11, C12, C13, C14, C2, C3, C4, C5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

Commit message: Changes in footprints, changed VCC pin in SX1308
+ changed polarized capacitors footprints to biiger ones
+ changed SX1308 footprint to 6 legged version
+ changed logic VCC for L293 from 3.3V to 5V
Parts:
- C1, C13, C15, C3, C6: footprint Capacitor_SMD:CP_Elec_5x4.4 -> Capacitor_SMD:CP_Elec_6.3x4.5
- U2: footprint Package_TO_SOT_SMD:SOT-23-5_HandSoldering -> Package_TO_SOT_SMD:SOT-23-6_Handsoldering
Connections:
- net at C15.1, C16.1, U10.8 (VCC2)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: now also R31.2, U10.1 (EN1,2), U10.16 (VCC1)
- now unconnected: J7.3 (Pin_3)
- no-connect marks 16 -> 17
Changed lines of the file:
@@
 F 0 "U2" H 3300 2125 50  0000 C CNN
 F 1 "SX1308" H 3300 2034 50  0000 C CNN
-F 2 "Package_TO_SOT_SMD:SOT-23-5_HandSoldering" H 3300 2100 50  0001 C CNN
+F 2 "Package_TO_SOT_SMD:SOT-23-6_Handsoldering" H 3300 2100 50  0001 C CNN
 F 3 "" H 3300 2100 50  0001 C CNN
 	1    3300 1700
@@
 F 0 "C6" H 5138 1546 50  0000 L CNN
 F 1 "47uF" H 5138 1455 50  0000 L CNN
-F 2 "Capacitor_SMD:CP_Elec_5x4.4" H 5050 1500 50  0001 C CNN
+F 2 "Capacitor_SMD:CP_Elec_6.3x4.5" H 5050 1500 50  0001 C CNN
 F 3 "~" H 5050 1500 50  0001 C CNN
 	1    5050 1500
@@
 F 0 "C1" H 1638 1396 50  0000 L CNN
 F 1 "47uF" H 1638 1305 50  0000 L CNN
-F 2 "Capacitor_SMD:CP_Elec_5x4.4" H 1550 1350 50  0001 C CNN
+F 2 "Capacitor_SMD:CP_Elec_6.3x4.5" H 1550 1350 50  0001 C CNN
 F 3 "~" H 1550 1350 50  0001 C CNN
 	1    1550 1350
@@
 F 0 "C3" H 3788 2946 50  0000 L CNN
 F 1 "47uF" H 3788 2855 50  0000 L CNN
-F 2 "Capacitor_SMD:CP_Elec_5x4.4" H 3700 2900 50  0001 C CNN
+F 2 "Capacitor_SMD:CP_Elec_6.3x4.5" H 3700 2900 50  0001 C CNN
 F 3 "~" H 3700 2900 50  0001 C CNN
 	1    3700 2900
@@
 U 1 1 5F1E3E2E
 P 2500 5300
-F 0 "U1" H 2300 6550 50  0000 C CNN
-F 1 "DS3231M" H 2300 6450 50  0000 C CNN
+F 0 "U1" H 1750 5050 50  0000 C CNN
+F 1 "DS3231M" H 1750 4950 50  0000 C CNN
 F 2 "Package_SO:SOIC-16W_7.5x10.3mm_P1.27mm" H 2500 4700 50  0001 C CNN
 F 3 "http://datasheets.maximintegrated.com/en/ds/DS3231.pdf" H 2770 5350 50  0001 C CNN
@@
 F 0 "C13" H 1488 7746 50  0000 L CNN
 F 1 "47uF" H 1488 7655 50  0000 L CNN
-F 2 "Capacitor_SMD:CP_Elec_5x4.4" H 1400 7700 50  0001 C CNN
+F 2 "Capacitor_SMD:CP_Elec_6.3x4.5" H 1400 7700 50  0001 C CNN
 F 3 "~" H 1400 7700 50  0001 C CNN
 	1    1400 7700
@@
 	6700 6200 6950 6200
 Wire Wire Line
-	10550 6200 10550 6550
-Wire Wire Line
 	7250 6500 7250 6550
 Wire Wire Line
@@
 	8950 7800 8950 6950
 Connection ~ 8950 7800
-Wire Wire Line
-	8850 7700 8850 6500
-Wire Wire Line
-	8850 6500 9550 6500
 Connection ~ 9800 6500
 Text Notes 6200 7550 2    50   ~ 0
@@
 	7550 6200 7700 6200
 Wire Wire Line
-	6450 7700 8850 7700
-Wire Wire Line
 	6450 7800 8950 7800
 Wire Wire Line
@@
 F 0 "C15" H 7788 6446 50  0000 L CNN
 F 1 "47uF" H 7788 6355 50  0000 L CNN
-F 2 "Capacitor_SMD:CP_Elec_5x4.4" H 7700 6400 50  0001 C CNN
+F 2 "Capacitor_SMD:CP_Elec_6.3x4.5" H 7700 6400 50  0001 C CNN
 F 3 "~" H 7700 6400 50  0001 C CNN
 	1    7700 6400
@@
 Connection ~ 8100 6200
 Wire Wire Line
-	8100 6200 10550 6200
-Wire Wire Line
 	8100 6500 8100 6550
 Wire Wire Line
@@
 Wire Wire Line
 	9550 6600 9550 6500
-Connection ~ 9550 6500
 Wire Wire Line
 	9550 6500 9800 6500
@@
 	9550 7150 9550 7600
 Connection ~ 9550 7150
+Wire Wire Line
+	8100 6200 10350 6200
+Wire Wire Line
+	10550 6500 10350 6500
+Wire Wire Line
+	10550 6500 10550 6550
+Connection ~ 10350 6500
+Wire Wire Line
+	10350 6500 10350 6200
+NoConn ~ 6450 7700
 $EndSCHEMATC
